File: Hardware/Analogue/ThePreamp-Analogue.kicad_sch (KiCad schematic)
At the start: 43 parts, among them J1 Replace, J2 Replace, J3 8V, J4 12V, J5 I2C, J6 SPI, J7 Conn_01x03_Female, J8 Conn_01x03_Female, J9 Conn_01x03_Female, K1 EA2-12NJ, K2 EA2-12NJ, K3 EA2-12NJ, K4 EA2-12NJ, U1 ULN2803ADWR, U2 MCP23008-E_SO, U3 Muses_72323

Commit message: update analogue schematic
Parts:
- added J1, J2: (no value), symbol Connector:Conn_01x02_Female
- added J5: (no value), symbol Connector_Generic:Conn_01x03
- C1: renamed from C2; value 100 uf/25V -> (none); footprint Capacitor_THT:CP_Radial_D8.0mm_P3.50mm -> (none)
- C2: renamed from C3; value 100 uf/25V -> (none); footprint Capacitor_THT:CP_Radial_D8.0mm_P3.50mm -> (none)
- C3: renamed from C4; value 10 uf/50V -> (none); footprint Capacitor_THT:CP_Radial_D8.0mm_P3.50mm -> (none)
- C4: renamed from C1; value 0.1uF -> (none); footprint Capacitor_SMD:C_0805_2012Metric_Pad1.15x1.40mm_HandSolder -> (none)
- C5, C7: value 100 uf/25V -> (none); footprint Capacitor_THT:CP_Radial_D8.0mm_P3.50mm -> (none)
- C6: value 0,1uF -> (none)
- J10: renamed from J7; value Conn_01x03_Female -> (none); footprint Connector_PinHeader_2.54mm:PinHeader_1x03_P2.54mm_Vertical -> (none)
- J11: renamed from J8; value Conn_01x03_Female -> (none); footprint Connector_PinHeader_2.54mm:PinHeader_1x03_P2.54mm_Vertical -> (none)
- J12: renamed from J9; value Conn_01x03_Female -> (none); footprint Connector_PinHeader_2.54mm:PinHeader_1x03_P2.54mm_Vertical -> (none)
- J13: renamed from J?; value ADS1115 -> (none)
- J14, J15, J3, J4: renamed from J?; value Conn_01x02_Female -> (none); footprint Connector_PinHeader_2.54mm:PinHeader_1x02_P2.54mm_Vertical -> (none)
- J16: renamed from J1; value Replace -> (none); footprint Connector_JST:JST_XH_B2B-XH-A_1x02_P2.50mm_Vertical -> (none)
- J17: renamed from J2; value Replace -> (none); footprint Connector_JST:JST_XH_B2B-XH-A_1x02_P2.50mm_Vertical -> (none)
- J6: renamed from J5; value I2C -> (none); footprint Connector_JST:JST_XH_B4B-XH-A_1x04_P2.50mm_Vertical -> (none)
- J7: renamed from J6; value SPI -> (none); footprint Connector_JST:JST_XH_B6B-XH-A_1x06_P2.50mm_Vertical -> (none)
- J8: renamed from J3; value 8V -> (none); footprint TerminalBlock:TerminalBlock_bornier-2_P5.08mm -> (none)
- J9: renamed from J4; value 12V -> (none); footprint TerminalBlock:TerminalBlock_bornier-2_P5.08mm -> (none)
- K1, K2, K3, K4: value EA2-12NJ -> (none)
- K5: renamed from K?; value EA2-12NJ -> (none)
- R1: renamed from R3; value 0 -> (none)
- R2: renamed from R4; value 10 -> (none)
- R3: renamed from R1; value 10K -> (none); footprint Resistor_SMD:R_0805_2012Metric_Pad1.15x1.40mm_HandSolder -> (none)
- R4: renamed from R2; value 10K -> (none); footprint Resistor_SMD:R_0805_2012Metric_Pad1.15x1.40mm_HandSolder -> (none)
- RCA1, RCA2, RCA3, RCA4, RCA5, RCA6, RCA7, RCA8: value RCA_Connector_ALI -> (none); footprint Connector_Audio:RCA Connector ALI -> (none)
- RCA10, RCA9: renamed from RCA?; value RCA_Connector_ALI -> (none); footprint Connector_Audio:RCA Connector ALI -> (none)
- U1: value ULN2803ADWR -> (none); footprint ULN2803:ULN2803ADWR -> (none)
- U2: renamed from U3; value Muses_72323 -> (none)
- U3: renamed from U2; value MCP23008-E_SO -> (none); footprint MCP23008:MCP23008-E&slash_SO -> (none)
Connections:
- net +8V is gone; now on net +3V3: J8.1 (Pin_1)
- net +12V: now also J9.1 (Pin_1)
- net +15V: now also J5.1 (Pin_1)
- net -15V: now also J5.3 (Pin_3)
- net Audio L: now also J1.1 (Pin_1); no longer J15.1 (Pin_1), K5.4
- net Audio R: now also J2.1 (Pin_1); no longer J14.1 (Pin_1), K5.7
- net GND: now also J14.2 (Pin_2), J15.2 (Pin_2), J3.2 (Pin_2), J4.2 (Pin_2), J9.2 (Pin_2), RCA10.2 (Ext), RCA9.2 (Ext), J1.2 (Pin_2), J2.2 (Pin_2), J5.2 (Pin_2)
- net GNDA: no longer RCA10.2 (Ext), RCA9.2 (Ext)
- net at RCA10.1 (In): now also K5.7; no longer K5.8
- net at RCA9.1 (In): now also K5.4; no longer K5.3
- new net Audio L out: J15.1 (Pin_1), K5.3
- new net Audio R out: J14.1 (Pin_1), K5.8
- no-connect marks 23 -> 24
Other:
- moved on the sheet: C1, C2, C3, C4, C5, C6, C7, J10, J11, J12, J13, J14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

Commit message: more pcb layout
Parts:
- removed C1, C2, C3, C5, C7: (no value), symbol Device:C_Polarized
- removed C6: (no value), symbol Device:C_Small
- removed J1, J14, J15, J2, J3, J4: (no value), symbol Connector:Conn_01x02_Female
- removed J10, J11, J12: (no value), symbol Connector:Conn_01x03_Female
- removed J5: (no value), symbol Connector_Generic:Conn_01x03
- removed J6: (no value), symbol Connector:Conn_01x04_Male
- removed J7: (no value), symbol Connector:Conn_01x06_Male
- removed J8, J9: (no value), symbol Connector_Generic:Conn_01x02
- removed U1: (no value), symbol Mezmerize_B1_Controller-rescue:ULN2803ADWR-2019-12-07_08-18-10
- removed U2: (no value), symbol muses72323:Muses_72323
- added IC1: ULN2803CDWR, SOIC127P1030X265-20N, symbol ULN2803:ULN2803CDWR
- added J1: To preamp, Connector_PinHeader_2.54mm:PinHeader_1x03_P2.54mm_Vertical, symbol Connector:Conn_01x03_Female
- added J2: From preamp, Connector_PinHeader_2.54mm:PinHeader_1x03_P2.54mm_Vertical, symbol Connector:Conn_01x03_Female
- added J3: Digital In, Connector_JST:JST_XH_B8B-XH-A_1x08_P2.50mm_Vertical, symbol Connector:Conn_01x08_Female
- added J4: Digital Pass Through, Connector_PinHeader_2.54mm:PinHeader_1x08_P2.54mm_Vertical, symbol Connector:Conn_01x08_Female
- added J5: Power In, Connector_JST:JST_XH_B5B-XH-A_1x05_P2.50mm_Vertical, symbol Connector:Conn_01x05_Female
- added J6: Power Out, Connector_PinHeader_2.54mm:PinHeader_1x05_P2.54mm_Vertical, symbol Connector:Conn_01x05_Female
- C1: renamed from C4; value (none) -> 0.1uF; footprint (none) -> Capacitor_SMD:C_0805_2012Metric_Pad1.18x1.45mm_HandSolder
- J7: renamed from J13; value (none) -> ADS1115; footprint (none) -> Connector_PinHeader_2.54mm:PinHeader_1x10_P2.54mm_Vertical
- J8: renamed from J16; value (none) -> Replace; footprint (none) -> Connector_JST:JST_XH_B2B-XH-A_1x02_P2.50mm_Vertical
- J9: renamed from J17; value (none) -> Replace; footprint (none) -> Connector_JST:JST_XH_B2B-XH-A_1x02_P2.50mm_Vertical
- K1: value (none) -> Input 1; footprint (none) -> EA2-12NJ:DIPS762W60P254L1420H630Q10N
- K2: value (none) -> Input 2; footprint (none) -> EA2-12NJ:DIPS762W60P254L1420H630Q10N
- K3: value (none) -> Input 3; footprint (none) -> EA2-12NJ:DIPS762W60P254L1420H630Q10N
- K4: value (none) -> Input 4; footprint (none) -> EA2-12NJ:DIPS762W60P254L1420H630Q10N
- K5: value (none) -> Output Mute; footprint (none) -> EA2-12NJ:DIPS762W60P254L1420H630Q10N
- R1, R2: value (none) -> 0R; footprint (none) -> Resistor_THT:R_Axial_DIN0207_L6.3mm_D2.5mm_P7.62mm_Horizontal
- R3, R4: value (none) -> 10K; footprint (none) -> Resistor_SMD:R_0805_2012Metric_Pad1.20x1.40mm_HandSolder
- RCA1, RCA10, RCA2, RCA3, RCA4, RCA5, RCA6, RCA7, RCA8, RCA9: value (none) -> RCA_Connector_ALI; footprint (none) -> Connector_Audio:RCA Connector ALI
- U1: renamed from U3; value (none) -> MCP23008-E_SO; footprint (none) -> MCP23008:SOIC127P1030X265-18N
Connections:
- net +12V: now also J5.4 (Pin_4), J6.4 (Pin_4)
- net +15V: now also J5.1 (Pin_1), J6.1 (Pin_1)
- net +3V3: now also J3.4 (Pin_4), J4.4 (Pin_4); no longer R2.2
- net -15V: now also J5.3 (Pin_3), J6.3 (Pin_3)
- net Audio L: now also R2.2, J1.3 (Pin_3)
- net Audio L out: now also R2.1, J2.3 (Pin_3)
- net Audio R: now also R1.2, J1.1 (Pin_1)
- net Audio R out: now also R1.1, J2.1 (Pin_1)
- net GND: now also IC1.9 (GND), J3.3 (Pin_3), J4.3 (Pin_3), J5.5 (Pin_5), J6.5 (Pin_5); no longer R1.1, RCA10.2 (Ext), RCA9.2 (Ext)
- net GNDA: now also RCA10.2 (Ext), RCA9.2 (Ext), J1.2 (Pin_2), J2.2 (Pin_2), J5.2 (Pin_2), J6.2 (Pin_2)
- net I2C:SCL: now also J3.2 (Pin_2), J4.2 (Pin_2)
- net I2C:SDA: now also J3.1 (Pin_1), J4.1 (Pin_1)
- net RELAY1: now also IC1.17 (4C); no longer K5.10
- net RELAY2: now also IC1.16 (5C)
- net RELAY3: now also IC1.15 (6C)
- net RELAY4: now also IC1.14 (7C)
- net RELAY5: now also K5.10, IC1.13 (8C)
- net SPI:MISO: now also J3.6 (Pin_6), J4.6 (Pin_6)
- net SPI:MOSI: now also J3.7 (Pin_7), J4.7 (Pin_7)
- net SPI:SCK: now also J3.5 (Pin_5), J4.5 (Pin_5)
- net SPI:SS: now also J3.8 (Pin_8), J4.8 (Pin_8)
- net at U1.17 (GP7): now also IC1.1 (1B)
- net at U1.16 (GP6): now also IC1.2 (2B)
- net at U1.15 (GP5): now also IC1.3 (3B)
- net at U1.14 (GP4): now also IC1.4 (4B)
- net at U1.13 (GP3): now also IC1.5 (5B)
- net at U1.12 (GP2): now also IC1.6 (6B)
- net at U1.11 (GP1): now also IC1.7 (7B)
- net at U1.10 (GP0): now also IC1.8 (8B)
- net A2: no longer names the net of J7.9 (Pin_9)
- net A3: no longer names the net of J7.10 (Pin_10)
- no-connect marks 24 -> 31
Other:
- moved on the sheet: C1, J7, J8, J9, K1, K2, K3, K4, K5, R3, R4, RCA1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
