File: Hardware/Analogue/ThePreamp-Analogue.kicad_pcb (KiCad board)
At the start: 2 copper layers, 240 x 65 mm, 37 parts, among them J1 Audio In Left, J10 Buffer Power, J11 Buffer In Left, J12 Buffer In Right, J13 ADS1115, J14 Buffer Out Right, J15 Buffer Out Left, J16 Replace, J17 Replace, J2 Audio In Right, J3 Audio In Right, J4 Audio In Left, J5 Audio Power, J6 I2C, J7 SPI, J8 Digital Power, J9 Relay Power, K1 Input 1, K2 Input 2, K3 Input 3, K4 Input 4, K5 Output Mute

Commit message: more pcb layout
Parts:
- removed C2, C5, C7: 100 uf/25V, Capacitor_THT:CP_Radial_D8.0mm_P3.50mm
- removed C3: 10 uf/50V, Capacitor_THT:CP_Radial_D8.0mm_P3.50mm
- removed J10: Buffer Power, Connector_PinHeader_2.54mm:PinHeader_1x03_P2.54mm_Vertical
- removed J11: Buffer In Left, Connector_PinHeader_2.54mm:PinHeader_1x03_P2.54mm_Vertical
- removed J12: Buffer In Right, Connector_PinHeader_2.54mm:PinHeader_1x03_P2.54mm_Vertical
- removed J14: Buffer Out Right, Connector_PinHeader_2.54mm:PinHeader_1x02_P2.54mm_Vertical
- removed J15: Buffer Out Left, Connector_PinHeader_2.54mm:PinHeader_1x02_P2.54mm_Vertical
- removed the J7 at (135.7, 22.2)
- removed the J8 at (202.9, 23.3)
- removed the J9 at (183.5, 38.4)
- added IC1: ULN2803CDWR, ULN2803:SOIC127P1030X265-20N, B.Cu at (29.2, 88.4)
- added R1: 0R, Resistor_THT:R_Axial_DIN0207_L6.3mm_D2.5mm_P7.62mm_Horizontal, B.Cu at (150.7, 100.5)
- added R2: 0R, Resistor_THT:R_Axial_DIN0207_L6.3mm_D2.5mm_P7.62mm_Horizontal, B.Cu at (150.6, 105.6)
- added R3: 10K, Resistor_SMD:R_0805_2012Metric_Pad1.20x1.40mm_HandSolder, B.Cu at (234.2, 132.2)
- added R4: 10K, Resistor_SMD:R_0805_2012Metric_Pad1.20x1.40mm_HandSolder, B.Cu at (234.1, 134.9)
- added REF**: MountingHole_3.2mm_M3, MountingHole:MountingHole_3.2mm_M3, F.Cu at (85.3, 79.6)
- added REF**: MountingHole_3.2mm_M3, MountingHole:MountingHole_3.2mm_M3, F.Cu at (215.3, 79.6)
- added REF**: MountingHole_3.2mm_M3, MountingHole:MountingHole_3.2mm_M3, F.Cu at (215.3, 134.6)
- added REF**: MountingHole_3.2mm_M3, MountingHole:MountingHole_3.2mm_M3, F.Cu at (85.3, 134.6)
- added U1: MCP23008-E_SO, MCP23008:SOIC127P1030X265-18N, B.Cu at (30.0, 102.5)
- C1: value 100 uf/25V -> 0.1uF; footprint Capacitor_THT:CP_Radial_D8.0mm_P3.50mm -> Capacitor_SMD:C_0805_2012Metric_Pad1.18x1.45mm_HandSolder; moved to B.Cu
- J1: value Audio In Left -> To preamp; footprint Connector_PinHeader_2.54mm:PinHeader_1x02_P2.54mm_Vertical -> Connector_PinHeader_2.54mm:PinHeader_1x03_P2.54mm_Vertical; moved to B.Cu
- J2: value Audio In Right -> From preamp; footprint Connector_PinHeader_2.54mm:PinHeader_1x02_P2.54mm_Vertical -> Connector_PinHeader_2.54mm:PinHeader_1x03_P2.54mm_Vertical; moved to B.Cu
- J3: value Audio In Right -> Digital In; footprint Connector_PinHeader_2.54mm:PinHeader_1x02_P2.54mm_Vertical -> Connector_JST:JST_XH_B8B-XH-A_1x08_P2.50mm_Vertical; moved to B.Cu
- J4: value Audio In Left -> Digital Pass Through; footprint Connector_PinHeader_2.54mm:PinHeader_1x02_P2.54mm_Vertical -> Connector_PinHeader_2.54mm:PinHeader_1x08_P2.54mm_Vertical; moved to B.Cu
- J5: value Audio Power -> Power In; footprint TerminalBlock:TerminalBlock_bornier-3_P5.08mm -> Connector_JST:JST_XH_B5B-XH-A_1x05_P2.50mm_Vertical; moved to B.Cu
- J6: value I2C -> Power Out; footprint Connector_JST:JST_XH_B4B-XH-A_1x04_P2.50mm_Vertical -> Connector_PinHeader_2.54mm:PinHeader_1x05_P2.54mm_Vertical; moved to B.Cu
- J7: renamed from J13; moved to B.Cu
- J8: renamed from J16; moved to B.Cu
- J9: renamed from J17; moved to B.Cu
- moved J7 190.8 mm to (226.9, 135.7)
- moved C1 175.7 mm to (29.7, 112.1)
- moved K5 173.4 mm to (243.5, 112.6), turned to 90 degrees
- moved J2 137.0 mm to (215.3, 100.6), turned to 180 degrees
- moved J5 84.9 mm to (25.9, 134.9)
- moved J3 80.0 mm to (55.9, 135.3)
- moved J9 79.9 mm to (235.2, 114.0), turned to 180 degrees
- moved J8 79.9 mm to (235.2, 124.0), turned to 180 degrees
- moved J4 70.5 mm to (85.3, 110.6), turned to 180 degrees
- moved J6 68.8 mm to (85.3, 85.6), turned to 180 degrees
- moved K4 60.7 mm to (118.7, 90.9), turned to 90 degrees
- moved J1 54.8 mm to (85.3, 100.6), turned to 180 degrees
- moved K2 50.8 mm to (67.7, 90.6), turned to 90 degrees
- moved K3 44.9 mm to (93.2, 91.1), turned to 90 degrees
- moved K1 21.4 mm to (42.2, 90.6), turned to 90 degrees
Connections:
- C1 pad 1: +15V -> +3V3
- J1 pad 1: Audio L -> Audio R
- J1 pad 2: GND -> GNDA
- J2 pad 1: Audio R -> Audio R out
- J2 pad 2: GND -> GNDA
- J3 pad 1: Audio R buffer -> I2C:SDA
- J3 pad 2: GND -> I2C:SCL
- J4 pad 1: Audio L buffer -> I2C:SDA
- J4 pad 2: GND -> I2C:SCL
- J5 pad 2: GND -> GNDA
- J6 pad 1: I2C:SCL -> +15V
- J6 pad 2: I2C:SDA -> GNDA
- J6 pad 3: GND -> -15V
- J6 pad 4: +3V3 -> +12V
- J7 pad 10: A3 -> unconnected-(J7-Pad10)
- J7 pad 9: A2 -> unconnected-(J7-Pad9)
- K5 pad 10: RELAY1 -> RELAY5
- RCA10 pad 2: GND -> GNDA
- RCA9 pad 2: GND -> GNDA
Routing:
- net +12V: track 0.00 -> 387.4 mm
- net GNDA: track 0.00 -> 386.1 mm
- net GND: track 0.00 -> 322.9 mm, vias 0 -> 5
- net +3V3: track 0.00 -> 274.1 mm
- net I2C:SDA: track 0.00 -> 246.6 mm
- net I2C:SCL: track 0.00 -> 242.8 mm
- net RELAY5: track 0.00 -> 233.7 mm
- net Audio L: track 0.00 -> 164.8 mm
- net Audio R: track 0.00 -> 161.1 mm
- net -15V: track 0.00 -> 120.5 mm
- net +15V: track 0.00 -> 114.6 mm
- net Audio R out: track 0.00 -> 101.3 mm
- net Audio L out: track 0.00 -> 100.9 mm
- net RELAY4: track 0.00 -> 99.0 mm
- net RELAY3: track 0.00 -> 70.9 mm
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Other:
- board text added: "Preamp pcb dim 140 x 65 mm Mounting holes 3.2 mm 5mm from edges"

Commit message: KiCad 7 and updated pcb
Parts:
- moved K3 0.50 mm to (93.2, 90.6)
- moved K4 0.30 mm to (118.7, 90.6)
Routing:
- net GNDA: track 386.1 -> 431.9 mm
- net Net-(IC1-Pad2): track 0.00 -> 5.16 mm
- net Net-(IC1-Pad1): track 0.00 -> 5.16 mm
- net +12V: track 387.4 -> 392.4 mm
- net GND: track 322.9 -> 325.7 mm
- net +3V3: track 274.1 -> 276.8 mm
- net Audio R: track 161.1 -> 163.0 mm
- net Audio L: track 164.8 -> 166.1 mm
- net Net-(K3-Pad3): track 28.7 -> 29.7 mm
- net Net-(K1-Pad3): track 28.8 -> 29.6 mm
- net Net-(K2-Pad3): track 28.8 -> 29.6 mm
- net Net-(K4-Pad3): track 28.9 -> 29.7 mm
- net I2C:SCL: track 242.8 -> 243.6 mm
- net RELAY4: track 99.0 -> 99.6 mm
- net Net-(K3-Pad8): track 18.0 -> 18.5 mm

Commit message: Cleanup
Routing:
- net GND: track 325.7 -> 331.1 mm, vias 5 -> 4
- net +12V: track 392.4 -> 389.2 mm
- net RELAY2: track 44.5 -> 41.6 mm
- net RELAY4: track 99.6 -> 97.4 mm
- net I2C:SDA: track 246.6 -> 244.5 mm
- net RELAY3: track 71.1 -> 69.1 mm
- net I2C:SCL: track 243.6 -> 242.1 mm
- net -15V: track 120.5 -> 119.7 mm
- net +3V3: track 276.8 -> 276.3 mm
