File: Hardware/Digital PSU/Digital PSU.kicad_pcb (KiCad board)
At the start: 2 copper layers, 241.4 x 87.4 mm, 51 parts, among them J1 AC in, J2 Relay power, J3 Conn_02x09, J4 15V AC, J5 230V AC, J6 ESP32 power, J7 Opt. 3V3 power, J8 DC in, J9 Relay power, Q1 NJW0302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

Commit message: Chassis placement new draft
Other:
- board text added: "TO-DO: Mounting holes on trafo pcb and L-adapter pcb + cut-outs to allow transistors to be mounted on bottom of chassis + copper fills + led wiring"
- board text removed: "TO-DO: Mounting holes on trafo pcb and L-adapter pcb + cut-outs to allow transistors to be mounted on bottom of chassis + copper fills"
Changed lines of the file:
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@@
 		(fp_arc
 			(start -14.45 -8.074396)
-			(mid -13.587327 -8.949835)
+			(mid -13.587327 -8.949836)
 			(end -12.7 -8.099396)
 			(stroke
@@
 		(fp_arc
 			(start -9.45 -8.125)
-			(mid -8.587327 -9.00044)
+			(mid -8.587328 -9.00044)
 			(end -7.7 -8.15)
 			(stroke
@@
 		(fp_arc
 			(start -9.45 -8.125)
-			(mid -8.587327 -9.00044)
+			(mid -8.587328 -9.00044)
 			(end -7.7 -8.15)
 			(stroke
@@
 		(fp_arc
 			(start -14.45 -8.074396)
-			(mid -13.587327 -8.949835)
+			(mid -13.587327 -8.949836)
 			(end -12.7 -8.099396)
 			(stroke
@@
 		(fp_arc
 			(start -14.45 -8.074396)
-			(mid -13.587327 -8.949828)
+			(mid -13.587327 -8.949829)
 			(end -12.7 -8.099396)
 			(stroke
@@
 		(fp_arc
 			(start -9.45 -8.125)
-			(mid -8.587327 -9.000433)
+			(mid -8.587327 -9.000434)
 			(end -7.7 -8.15)
 			(stroke
@@
 		(fp_arc
 			(start -14.45 -8.074396)
-			(mid -13.587327 -8.949828)
+			(mid -13.587327 -8.949829)
 			(end -12.7 -8.099396)
 			(stroke
@@
 		(fp_arc
 			(start -9.45 -8.125)
-			(mid -8.587327 -9.000433)
+			(mid -8.587327 -9.000434)
 			(end -7.7 -8.15)
 			(stroke
@@
 		(fp_arc
 			(start -9.45 -8.125)
-			(mid -8.587327 -9.00044)
+			(mid -8.587328 -9.00044)
 			(end -7.7 -8.15)
 			(stroke
@@
 		(fp_arc
 			(start -14.45 -8.074396)
-			(mid -13.587327 -8.949835)
+			(mid -13.587327 -8.949836)
 			(end -12.7 -8.099396)
 			(stroke
@@
 		(fp_arc
 			(start -14.45 -8.074396)
-			(mid -13.587327 -8.949835)
+			(mid -13.587327 -8.949836)
 			(end -12.7 -8.099396)
 			(stroke
@@
 		(fp_arc
 			(start -9.45 -8.125)
-			(mid -8.587327 -9.00044)
+			(mid -8.587328 -9.00044)
 			(end -7.7 -8.15)
 			(stroke
@@
 		(layer "Edge.Cuts")
 	)
-	(gr_text "TO-DO: Mounting holes on trafo pcb and L-adapter pcb + cut-outs to allow transistors to be mounted on bottom of chassis + copper fills"
+	(gr_rect
+		(start 20.34 24.63)
+		(end 102.58 112.06)
+		(stroke
+			(width 0.2)
+			(type default)
+		)
+		(fill none)
+		(layer "F.Fab")
+	)
+	(gr_text "TO-DO: Mounting holes on trafo pcb and L-adapter pcb + cut-outs to allow transistors to be mounted on bottom of chassis + copper fills + led wiring"
 		(at 44.88 110.81 0)
 		(layer "F.SilkS")

Commit message: Chassis placement draft
Parts:
- J6: value ESP32 power -> 8V
- J7: value Opt. 3V3 power -> Opt. 3V3
- J9: value Relay power -> 12V
- moved J9 66.0 mm to (271.7, 100.7), turned to 180 degrees
- moved J6 40.2 mm to (259.1, 100.7), turned to 180 degrees
- moved HS7 26.7 mm to (248.7, 71.2), turned to 180 degrees
- moved U3 23.8 mm to (246.2, 74.7), turned to 0 degrees
- moved C8 18.9 mm to (245.7, 79.5), turned to 180 degrees
- moved HS6 15.4 mm to (248.8, 53.5), turned to 180 degrees
- moved C6 14.0 mm to (252.2, 79.5), turned to 180 degrees
- moved U2 10.8 mm to (246.3, 57.0), turned to 0 degrees
- moved J7 9.16 mm to (246.5, 100.7), turned to 180 degrees
- moved C7 7.11 mm to (252.6, 61.7), turned to 180 degrees
- moved C5 4.97 mm to (246.0, 61.7), turned to 180 degrees
- moved J2 4.47 mm to (221.2, 37.9)
- moved J8 4.40 mm to (242.2, 42.9)
- moved D11 0.07 mm to (192.7, 38.5)
- moved D10 0.05 mm to (195.2, 38.5)
Routing:
- net +12V: track 178.0 -> 220.5 mm
- net Net-(D14-K): track 0.00 -> 7.03 mm
- net Net-(D12-K): track 0.00 -> 7.03 mm
- net Net-(D11-K): track 0.00 -> 7.02 mm
- net Net-(D10-K): track 0.00 -> 7.02 mm
- net Net-(D10-A): track 0.00 -> 7.02 mm
- net Net-(D7-K): track 0.00 -> 7.02 mm
- net Net-(D8-K): track 0.00 -> 7.01 mm
- net Net-(D6-K): track 0.00 -> 7.01 mm
- net Net-(D13-K): track 0.00 -> 7.01 mm
- net Net-(D15-K): track 42.3 -> 40.4 mm
Other:
- board size 241.4 x 87.4 mm -> 178.2 x 85 mm
- board text added: "TO-DO: Mounting holes on trafo pcb and L-adapter pcb + cut-outs to allow transistors to be mounted on bottom of chassis + copper fills"
- board text removed: "TO-DO: Mounting holes on trafo pcb and L-adapter pcb + cut-outs to allow transistors to be mounted on bottom of chassis + copper fills + led wiring"

Commit message: Small adjustments to draft
Parts:
- added H1: MountingHole, MountingHole:MountingHole_3.2mm_M3_DIN965, F.Cu at (26.1, 105.7)
- added H10: MountingHole, MountingHole:MountingHole_3.2mm_M3_DIN965, F.Cu at (236.1, 106.5)
- added H11: MountingHole, MountingHole:MountingHole_3.2mm_M3_DIN965, F.Cu at (281.4, 31.1)
- added H12: MountingHole, MountingHole:MountingHole_3.2mm_M3_DIN965, F.Cu at (281.7, 106.8)
- added H2: MountingHole, MountingHole:MountingHole_3.2mm_M3_DIN965, F.Cu at (98.4, 106.1)
- added H3: MountingHole, MountingHole:MountingHole_3.2mm_M3_DIN965, F.Cu at (25.8, 31.0)
- added H4: MountingHole, MountingHole:MountingHole_3.2mm_M3_DIN965, F.Cu at (98.5, 31.1)
- added H5: MountingHole, MountingHole:MountingHole_3.2mm_M3_DIN965, F.Cu at (108.6, 31.2)
- added H6: MountingHole, MountingHole:MountingHole_3.2mm_M3_DIN965, F.Cu at (108.6, 106.2)
- added H7: MountingHole, MountingHole:MountingHole_3.2mm_M3_DIN965, F.Cu at (226.8, 31.1)
- added H8: MountingHole, MountingHole:MountingHole_3.2mm_M3_DIN965, F.Cu at (226.4, 106.5)
- added H9: MountingHole, MountingHole:MountingHole_3.2mm_M3_DIN965, F.Cu at (236.6, 31.0)
- C5, C6, C7: moved to B.Cu
- J6: value 8V -> ESP32 power
- J7: value Opt. 3V3 -> Opt. 3V3 power
- J9: value 12V -> Relay power
- moved U2 29.4 mm to (256.2, 84.7)
- moved HS6 29.4 mm to (258.8, 81.2)
- moved C7 27.8 mm to (263.0, 87.5), turned to 0 degrees
- moved C6 23.7 mm to (253.7, 55.9)
- moved U3 20.6 mm to (261.2, 60.7), turned to 180 degrees
- moved C5 19.6 mm to (254.2, 79.5)
- moved C8 18.4 mm to (260.4, 68.5), turned to 0 degrees
- moved HS7 12.2 mm to (258.7, 64.2), turned to 0 degrees
- moved J7 2.28 mm to (248.8, 100.6)
- moved J6 2.28 mm to (261.4, 100.6)
- moved J9 2.28 mm to (274.0, 100.6)
- moved F2 0.90 mm to (26.4, 75.3)
- moved J4 0.90 mm to (93.2, 66.2)
- moved TR1 0.90 mm to (46.7, 83.8)
- moved J5 0.90 mm to (31.6, 56.3)
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Routing:
- net Net-(J7-Pin_1): track 0.00 -> 44.0 mm
- net +12V: track 220.5 -> 239.0 mm
- net Net-(J6-Pin_1): track 0.00 -> 16.0 mm
Other:
- board size 178.2 x 85 mm -> 265 x 85 mm
