File: Hardware/Digital PSU - 8V_3.3V/Digital PSU - 8V_3.3V.kicad_pcb (KiCad board)
At the start: 2 copper layers, 54.4 x 85 mm, 16 parts, among them J6 ESP32 power, J7 Opt. 3V3 power, J8 DC in, J9 Relay power, U2 LM7808_TO220, U3 LD1117V33

Commit message: Updated pcb 3.3V + adjust of connectors on controller pcb
Parts:
- C6: moved to F.Cu
- C8: moved to B.Cu
- moved C6 17.6 mm to (257.5, 71.0), turned to 0 degrees
Connections:
- C6 pad 1: +12V -> Net-(J6-Pin_1)
- U3 pad 3: +12V -> Net-(J6-Pin_1)
Routing:
- net Net-(J6-Pin_1): track 16.0 -> 42.1 mm
- net +12V: track 148.6 -> 128.2 mm
Other:
- board text added: "+12V"
- board text added: "+3.3V"
- board text added: "+8V"

Commit message: Last changes before ordering of pcb
Other:
- board text added: "LD1117V33"
- board text added: "LM7808 - LM78XX"
Changed lines of the file:
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@@
 		(tags "capacitor handsolder")
 		(property "Reference" "C6"
-			(at 0 -1.68 360)
+			(at 0 -1.68 0)
 			(layer "F.SilkS")
 			(hide yes)
@@
 		)
 		(property "Value" "100nF"
-			(at 0 1.68 360)
+			(at 0 1.68 0)
 			(layer "F.Fab")
 			(effects
@@
 		)
 		(fp_text user "${REFERENCE}"
-			(at 0 0 360)
+			(at 0 0 0)
 			(layer "F.Fab")
 			(effects
@@
 		(fp_arc
 			(start -14.45 -8.074396)
-			(mid -13.587327 -8.949835)
+			(mid -13.587327 -8.949836)
 			(end -12.7 -8.099396)
 			(stroke
@@
 		(fp_arc
 			(start -9.45 -8.125)
-			(mid -8.587327 -9.00044)
+			(mid -8.587328 -9.00044)
 			(end -7.7 -8.15)
 			(stroke
@@
 		(fp_arc
 			(start -9.45 -8.125)
-			(mid -8.587327 -9.00044)
+			(mid -8.587328 -9.00044)
 			(end -7.7 -8.15)
 			(stroke
@@
 		(fp_arc
 			(start -14.45 -8.074396)
-			(mid -13.587327 -8.949835)
+			(mid -13.587327 -8.949836)
 			(end -12.7 -8.099396)
 			(stroke
@@
 		(tags "capacitor handsolder")
 		(property "Reference" "C8"
-			(at 0 1.85 360)
+			(at 0 1.85 0)
 			(layer "B.SilkS")
 			(hide yes)
@@
 		)
 		(property "Value" "10uF 16V"
-			(at 0 -1.85 360)
+			(at 0 -1.85 0)
 			(layer "B.Fab")
 			(effects
@@
 		)
 		(fp_text user "${REFERENCE}"
-			(at 0 0 360)
+			(at 0 0 0)
 			(layer "B.Fab")
 			(effects
@@
 		)
 	)
+	(gr_text "LD1117V33"
+		(at 249.3 58.5 0)
+		(layer "F.SilkS")
+		(effects
+			(font
+				(size 1 1)
+				(thickness 0.1)
+			)
+			(justify left bottom)
+		)
+	)
 	(gr_text "+12V"
 		(at 240 38.5 0)
 		(layer "F.SilkS")
 		(effects
+			(font
+				(size 1 1)
+				(thickness 0.1)
+			)
+			(justify left bottom)
+		)
+	)
+	(gr_text "LM7808 - LM78XX"
+		(at 246.3 87.9 0)
+		(layer "F.SilkS")
+		(effects
