File: Hardware/Digital PSU - LAdapter/Digital PSU - LAdapter.kicad_pcb (KiCad board)
At the start: 2 copper layers, 128 x 85 mm, 39 parts, among them J1 AC in, J2 Relay power, J3 Conn_02x09, Q1 NJW0302, Q2 MJE15030, U1 LM334Z

Commit message: Last changes before ordering of pcb
Routing:
- added copper zone on B.Cu, net GND
Other:
- board text added: "+"
- board text added: "AC IN"
- board text added: "DC OUT"
- board text removed: "TO-DO: Mounting holes on trafo pcb and L-adapter pcb + cut-outs to allow transistors to be mounted on bottom of chassis + copper fills"
Changed lines of the file:
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@@
 		)
 		(property "Value" "~"
-			(at 1.27 2.06 -90)
+			(at 0.192916 1.815 -90)
 			(layer "F.Fab")
+			(hide yes)
 			(effects
 				(font
@@
 			(at 0 -3.8 0)
 			(layer "F.SilkS")
+			(hide yes)
 			(effects
 				(font
@@
 	(footprint "LED_THT:LED_Rectangular_W5.0mm_H2.0mm"
 		(layer "F.Cu")
-		(at 182.31 38.48 90)
+		(at 182.31 38.492916 90)
 		(descr "LED_Rectangular, Rectangular,  Rectangular size 5.0x2.0mm^2, 2 pins, http://www.kingbright.com/attachments/file/psearch/000/00/00/L-169XCGDK(Ver.9B).pdf")
 		(tags "LED_Rectangular Rectangular  Rectangular size 5.0x2.0mm^2 2 pins")
@@
 		(tags "TO-220-2 Vertical RM 5.08mm")
 		(property "Reference" "D4"
-			(at 2.54 -4.27 0)
+			(at 9.035 -0.647916 0)
 			(layer "F.SilkS")
 			(effects
@@
 		(tags "Resistor Axial_DIN0207 series Axial Horizontal pin pitch 10.16mm 0.25W = 1/4W length 6.3mm diameter 2.5mm")
 		(property "Reference" "R2"
-			(at 5.08 -2.37 0)
+			(at -2.435 -0.102916 0)
 			(layer "F.SilkS")
 			(effects
@@
 			(at 0 -3.8 0)
 			(layer "F.SilkS")
+			(hide yes)
 			(effects
 				(font
@@
 		(tags "heatsink fischer")
 		(property "Reference" "HS1"
-			(at -0.5 6.8 0)
+			(at 0.055 -1.471346 0)
 			(layer "F.SilkS")
+			(hide yes)
 			(effects
 				(font
@@
 		(tags "Resistor Axial_DIN0414 series Axial Horizontal pin pitch 15.24mm 2W length 11.9mm diameter 4.5mm")
 		(property "Reference" "R4"
-			(at 7.62 -3.37 180)
+			(at 3.225 3.412916 180)
 			(layer "F.SilkS")
 			(effects
@@
 	(footprint "LED_THT:LED_Rectangular_W5.0mm_H2.0mm"
 		(layer "F.Cu")
-		(at 187.39 38.49 90)
+		(at 187.39 38.492916 90)
 		(descr "LED_Rectangular, Rectangular,  Rectangular size 5.0x2.0mm^2, 2 pins, http://www.kingbright.com/attachments/file/psearch/000/00/00/L-169XCGDK(Ver.9B).pdf")
 		(tags "LED_Rectangular Rectangular  Rectangular size 5.0x2.0mm^2 2 pins")
@@
 		(tags "Resistor Axial_DIN0207 series Axial Horizontal pin pitch 10.16mm 0.25W = 1/4W length 6.3mm diameter 2.5mm")
 		(property "Reference" "R1"
-			(at 5.08 -2.37 0)
+			(at -2.525 -0.202916 0)
 			(layer "F.SilkS")
 			(effects
@@
 			(at -0.5 6.8 180)
 			(layer "F.SilkS")
+			(hide yes)
 			(effects
 				(font
@@
 			(at -0.5 6.8 180)
 			(layer "F.SilkS")
+			(hide yes)
 			(effects
 				(font
@@
 			(at 0 -3.8 0)
 			(layer "F.SilkS")
+			(hide yes)
 			(effects
 				(font
@@
 	(footprint "LED_THT:LED_Rectangular_W5.0mm_H2.0mm"
 		(layer "F.Cu")
-		(at 189.93 38.49 90)
+		(at 189.93 38.492916 90)
 		(descr "LED_Rectangular, Rectangular,  Rectangular size 5.0x2.0mm^2, 2 pins, http://www.kingbright.com/attachments/file/psearch/000/00/00/L-169XCGDK(Ver.9B).pdf")
 		(tags "LED_Rectangular Rectangular  Rectangular size 5.0x2.0mm^2 2 pins")
@@
 		(tags "Diode DO-41_SOD81 series Axial Horizontal pin pitch 7.62mm  length 5.2mm diameter 2.7mm")
 		(property "Reference" "D5"
-			(at 3.81 -2.47 0)
+			(at 3.81 2.647084 0)
 			(layer "F.SilkS")
 			(effects
@@
 		(tags "TO-220-2 Vertical RM 5.08mm")
 		(property "Reference" "D3"
-			(at 2.54 -4.27 0)
+			(at 9.115 -0.812916 0)
 			(layer "F.SilkS")
 			(effects
@@
 		(tags "TO-220-2 Vertical RM 5.08mm")
 		(property "Reference" "D1"
-			(at 2.54 -4.27 180)
+			(at -4.145 -1.187084 180)
 			(layer "F.SilkS")
 			(effects
@@
 		(tags "TO-220-2 Vertical RM 5.08mm")
 		(property "Reference" "D2"
-			(at 2.54 -4.27 180)
+			(at -4.135 -0.867084 180)
 			(layer "F.SilkS")
 			(effects
@@
 	(footprint "LED_THT:LED_Rectangular_W5.0mm_H2.0mm"
 		(layer "F.Cu")
-		(at 184.855 38.487916 90)
+		(at 184.855 38.492916 90)
 		(descr "LED_Rectangular, Rectangular,  Rectangular size 5.0x2.0mm^2, 2 pins, http://www.kingbright.com/attachments/file/psearch/000/00/00/L-169XCGDK(Ver.9B).pdf")
 		(tags "LED_Rectangular Rectangular  Rectangular size 5.0x2.0mm^2 2 pins")
@@
 		(tags "Potentiometer vertical Bourns 3296W")
 		(property "Reference" "R3"
-			(at -2.54 -3.66 90)
+			(at 3.257084 -0.095 180)
 			(layer "F.SilkS")
 			(effects
@@
 			(at 0 -3.8 0)
 			(layer "F.SilkS")
+			(hide yes)
 			(effects
 				(font
@@
 			(at -10.495 -2.772916 180)
 			(layer "F.SilkS")
+			(hide yes)
 			(effects
 				(font
@@
 		(tags "heatsink fischer")
 		(property "Reference" "HS3"
-			(at -0.5 6.8 0)
+			(at 0.295 -1.291346 0)
 			(layer "F.SilkS")
+			(hide yes)
 			(effects
 				(font
@@
 		(tags "CP Radial series Radial pin pitch 5.00mm  diameter 10mm Electrolytic Capacitor")
 		(property "Reference" "C4"
-			(at 2.5 -6.25 180)
+			(at 7.892677 -3.887084 180)
 			(layer "F.SilkS")
 			(effects
@@
 	(footprint "LED_THT:LED_Rectangular_W5.0mm_H2.0mm"
 		(layer "F.Cu")
-		(at 197.55 38.49 90)
+		(at 197.55 38.492916 90)
 		(descr "LED_Rectangular, Rectangular,  Rectangular size 5.0x2.0mm^2, 2 pins, http://www.kingbright.com/attachments/file/psearch/000/00/00/L-169XCGDK(Ver.9B).pdf")
 		(tags "LED_Rectangular Rectangular  Rectangular size 5.0x2.0mm^2 2 pins")
@@
 	(footprint "LED_THT:LED_Rectangular_W5.0mm_H2.0mm"
 		(layer "F.Cu")
-		(at 177.235 38.487916 90)
+		(at 177.235 38.492916 90)
 		(descr "LED_Rectangular, Rectangular,  Rectangular size 5.0x2.0mm^2, 2 pins, http://www.kingbright.com/attachments/file/psearch/000/00/00/L-169XCGDK(Ver.9B).pdf")
 		(tags "LED_Rectangular Rectangular  Rectangular size 5.0x2.0mm^2 2 pins")
@@
 		(layer "Edge.Cuts")
 	)
-	(gr_text "TO-DO: Mounting holes on trafo pcb and L-adapter pcb + cut-outs to allow transistors to be mounted on bottom of chassis + copper fills"
-		(at 39.62 110.78 0)
+	(gr_text "+"
+		(at 211.9 38.8 0)
+		(layer "F.SilkS")
+		(effects
+			(font
+				(size 1.5 1.5)
+				(thickness 0.3)
+				(bold yes)
+			)
+			(justify left bottom)
+		)
+	)
+	(gr_text "AC IN"
+		(at 102.2 61.7 0)
+		(layer "F.SilkS")
+		(effects
+			(font
+				(size 1.5 1.5)
+				(thickness 0.3)
+				(bold yes)
+			)
+			(justify left bottom)
+		)
+	)
+	(gr_text "DC OUT"
+		(at 215.4 49.1 0)
 		(layer "F.SilkS")
 		(effects
@@
 	)
 	(segment
-		(start 208.595 58.502916)
-		(end 208.595 58.445)
-		(width 3)
-		(layer "B.Cu")
-		(net 2)
-	)
-	(segment
-		(start 208.595 58.445)
-		(end 208.685 58.445)
-		(width 3)
-		(layer "B.Cu")
-		(net 2)
-	)
-	(segment
 		(start 208.595 45.2675)
 		(end 215.9825 37.88)
@@
 		(net 19)
 	)
+	(zone
+		(net 7)
+		(net_name "GND")
+		(layer "B.Cu")
+		(hatch edge 0.5)
+		(connect_pads
+			(clearance 0.5)
+		)
+		(min_thickness 0.25)
+		(filled_areas_thickness no)
+		(fill yes
+			(thermal_gap 0.5)
+			(thermal_bridge_width 0.5)
+		)
+		(polygon
+			(pts
+				(xy 98.4 26.1) (xy 226.2 26.1) (xy 226.2 110.9) (xy 98.663205 110.859087) (xy 98.5 110.9)
+			)
+		)
+	)
 )
