File: Hardware/Analogue/Buffer-Opamp/Buffer-Opamp.kicad_sch (KiCad schematic)
At the start: 21 parts

Commit message: analogue pcb work
Parts:
- C1, C2: renamed from C?; value 10 uF -> (none)
- C3, C4: renamed from C?; value 10 pF -> (none)
- C5, C6, C7, C8: renamed from C?; value 100 uf/25V -> (none); footprint Capacitor_THT:CP_Radial_D8.0mm_P3.50mm -> (none)
- J1, J2, J3: renamed from J?; value Conn_01x03_Female -> (none); footprint Connector_PinHeader_2.54mm:PinHeader_1x03_P2.54mm_Vertical -> (none)
- J4, J5: renamed from J?; value Conn_01x02_Female -> (none); footprint Connector_PinHeader_2.54mm:PinHeader_1x02_P2.54mm_Vertical -> (none)
- R1, R2: renamed from R?; value 100K -> (none)
- R3, R4: renamed from R?; value 47 -> (none)
- RV1, RV2: renamed from RV?; value 100k -> (none)
- U1, U2: renamed from U?; value NE5534 -> (none)
Connections:
- net GND: now also J4.2 (Pin_2)

Commit message: Separating digital and analog ground
Parts:
- C1, C2: value (none) -> 10 uF; footprint (none) -> Capacitor_THT:CP_Radial_D6.3mm_P2.50mm
- C3, C4: value (none) -> 10 pF; footprint (none) -> Capacitor_THT:C_Disc_D4.3mm_W1.9mm_P5.00mm
- C5, C6, C7, C8: value (none) -> 100 uf/25V; footprint (none) -> Capacitor_THT:CP_Radial_D8.0mm_P3.50mm
- J1, J2, J3: value (none) -> Conn_01x03_Female; footprint (none) -> Connector_PinHeader_2.54mm:PinHeader_1x03_P2.54mm_Vertical
- J4, J5: value (none) -> Conn_01x02_Female; footprint (none) -> Connector_PinHeader_2.54mm:PinHeader_1x02_P2.54mm_Vertical
- R1, R2: value (none) -> 100K; footprint (none) -> Resistor_THT:R_Axial_DIN0207_L6.3mm_D2.5mm_P10.16mm_Horizontal
- R3, R4: value (none) -> 47; footprint (none) -> Resistor_THT:R_Axial_DIN0207_L6.3mm_D2.5mm_P10.16mm_Horizontal
- RV1, RV2: value (none) -> 100k; footprint (none) -> Potentiometer_THT:Potentiometer_Bourns_3296W_Vertical
- U1, U2: value (none) -> NE5534; footprint (none) -> Package_DIP:DIP-8_W7.62mm_Socket_LongPads
