File: Hardware/Controller/ThePreamp-Controller.kicad_pcb (KiCad board)
At the start: 2 copper layers, 335.9 x 44.5 mm, 29 parts, among them J1 8V, J2 Power relay trigger, J3 SPI DISPLAY 1, J4 SPI DISPLAY 2, J5 Digital Out, J6 3.3V (Opt), J8 12V, SW1 RotaryEncoder_Switch, SW2 RotaryEncoder_Switch, U1 TSOP34838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

Commit message: Last changes before ordering of pcb
Routing:
- net SPI:SS_MUSES: track 146.3 -> 145.3 mm
Changed lines of the file:
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@@
 			)
 		)
-		(property "Footprint" ""
+		(property "Footprint" "MountingHole:MountingHole_3.2mm_M3_ISO7380"
 			(at 0 0 180)
 			(unlocked yes)
@@
 			)
 		)
-		(property "Footprint" ""
+		(property "Footprint" "MountingHole:MountingHole_3.2mm_M3_ISO7380"
 			(at 0 0 180)
 			(unlocked yes)
@@
 			)
 		)
-		(property "Footprint" ""
+		(property "Footprint" "MountingHole:MountingHole_3.2mm_M3_ISO7380"
 			(at 0 0 180)
 			(unlocked yes)
@@
 			)
 		)
-		(property "Footprint" ""
+		(property "Footprint" "MountingHole:MountingHole_3.2mm_M3_ISO7380"
 			(at 0 0 180)
 			(unlocked yes)
@@
 			)
 		)
-		(property "Footprint" ""
+		(property "Footprint" "MountingHole:MountingHole_3.2mm_M3_ISO7380"
 			(at 0 0 180)
 			(unlocked yes)
@@
 			)
 		)
-		(property "Footprint" ""
+		(property "Footprint" "MountingHole:MountingHole_3.2mm_M3_ISO7380"
 			(at 0 0 180)
 			(unlocked yes)
@@
 			)
 		)
-		(property "Footprint" "APC_817B1_SL:APC-817xx-SL_AMB-M"
+		(property "Footprint" "Package_DIP:DIP-4_W7.62mm"
 			(at 0 0 90)
 			(unlocked yes)
@@
 			)
 		)
-		(property "Footprint" ""
+		(property "Footprint" "The PreAmp logo:The PreAmp logo"
 			(at 0 0 180)
 			(unlocked yes)
@@
 			)
 		)
-		(property "Footprint" "MODULE_ESP32_DEVKIT_V1"
+		(property "Footprint" "ESP32FP:MODULE_ESP32_DEVKIT_V1"
 			(at 0 0 90)
 			(unlocked yes)
@@
 		(width 0.4)
 		(layer "F.Cu")
-		(net 17)
-	)
-	(segment
-		(start 272.49 51.82)
-		(end 273.455584 51.82)
-		(width 0.4)
-		(layer "F.Cu")

Commit message: Added pullup resistors on D34-35 on controller pcb
Parts:
- added R4: 10K, Resistor_SMD:R_0805_2012Metric_Pad1.20x1.40mm_HandSolder, B.Cu at (221.4, 70.8)
- added R5: 10K, Resistor_SMD:R_0805_2012Metric_Pad1.20x1.40mm_HandSolder, B.Cu at (218.9, 70.8)
- U4: footprint Package_DIP:DIP-4_W7.62mm -> APC_817B1_SL:APC-817xx-SL_AMB-M
Routing:
- net +3V3 ESP32: track 25.2 -> 65.1 mm
- net SW_1: track 46.8 -> 52.3 mm
- net SW_2: track 197.2 -> 202.7 mm

Commit message: Added 10uF for EN pin to stabilize init of displays
Parts:
- added C7: 10uF, Capacitor_THT:CP_Radial_D5.0mm_P2.50mm, B.Cu at (245.8, 82.3)
- moved C6 4.70 mm to (238.4, 84.0)
Connections:
- U3 pad 16: unconnected-(U3-EN-Pad16) -> Net-(U3-EN)
Routing:
- net Net-(U3-EN): track 0.00 -> 20.0 mm
- net +8V: track 97.5 -> 99.6 mm
